Commit message: debug the error

File: yahboomcar_ws/install/test_config/share/test_config/config/dofbot_pro_descripton.ros2_control.xacro (robot description, xacro)
@@ -1 +1,54 @@
-/home/pawan/yahboomcar_ws/src/test_config/config/dofbot_pro_descripton.ros2_control.xacro
+<?xml version="1.0"?>
+<robot xmlns:xacro="http://www.ros.org/wiki/xacro">
+    <xacro:macro name="dofbot_pro_descripton_ros2_control" params="name initial_positions_file">
+        <xacro:property name="initial_positions" value="${load_yaml(initial_positions_file)['initial_positions']}"/>
+        <ros2_control name="${name}" type="system">
+            <hardware>
+                <!-- By default, set up controllers for simulation. This won't work on real hardware -->
+                <plugin>mock_components/GenericSystem</plugin>
+            </hardware>
+            <joint name="arm1_Joint">
+                <command_interface name="position"/>
+                <state_interface name="position">
+                  <param name="initial_value">${initial_positions['arm1_Joint']}</param>
+                </state_interface>
+                <state_interface name="velocity"/>
+            </joint>
+            <joint name="arm2_Joint">
+                <command_interface name="position"/>
+                <state_interface name="position">
+                  <param name="initial_value">${initial_positions['arm2_Joint']}</param>
+                </state_interface>
+                <state_interface name="velocity"/>
+            </joint>
+            <joint name="arm3_Joint">
+                <command_interface name="position"/>
+                <state_interface name="position">
+                  <param name="initial_value">${initial_positions['arm3_Joint']}</param>
+                </state_interface>
+                <state_interface name="velocity"/>
+            </joint>
+            <joint name="arm4_Joiint">
+                <command_interface name="position"/>
+                <state_interface name="position">
+                  <param name="initial_value">${initial_positions['arm4_Joiint']}</param>
+                </state_interface>
+                <state_interface name="velocity"/>
+            </joint>
+            <joint name="arm5_Joint">
+                <command_interface name="position"/>
+                <state_interface name="position">
+                  <param name="initial_value">${initial_positions['arm5_Joint']}</param>
+                </state_interface>
+                <state_interface name="velocity"/>
+            </joint>
+            <joint name="rlink1_Joint">
+                <command_interface name="position"/>
+                <state_interface name="position">
+                  <param name="initial_value">${initial_positions['rlink1_Joint']}</param>
+                </state_interface>
+                <state_interface name="velocity"/>
+            </joint>
+        </ros2_control>
+    </xacro:macro>
+</robot>

File: yahboomcar_ws/install/test_config/share/test_config/config/dofbot_pro_descripton.urdf.xacro (robot description, xacro)
@@ -1 +1,9 @@
-/home/pawan/yahboomcar_ws/src/test_config/config/dofbot_pro_descripton.urdf.xacro
+<?xml version="1.0"?>
+<robot xmlns:xacro="http://www.ros.org/wiki/xacro" name="dofbot_pro_descripton">
+    <xacro:arg name="initial_positions_file" default="initial_positions.yaml" />
+    <!-- Import dofbot_pro_descripton urdf file -->
+    <xacro:include filename="$(find dofbot_pro_descripton)/urdf/X5PLUS_V12.urdf" />
+    <!-- Import control_xacro -->
+    <xacro:include filename="dofbot_pro_descripton.ros2_control.xacro" />
+    <xacro:dofbot_pro_descripton_ros2_control name="FakeSystem" initial_positions_file="$(arg initial_positions_file)"/>
+</robot>

File: yahboomcar_ws/install/yahboom_M3Pro_description/share/yahboom_M3Pro_description/urdf/M3Pro.urdf (robot description, URDF)
Before this commit: robot M3Pro, 20 links, 19 joints
Links:
- link arm_base_Link: geometry collision mesh filename=package://yahboom_M3Pro_description/meshes/arm_base_Link.STL; visual mesh filename=package://yahboom_M3Pro_description/meshes/arm_base_Link.STL
