Commit message: added Gazebo and rsp

File: yahboomcar_ws/src/yahboom_M3Pro_description/urdf/M3Pro.urdf (robot description, URDF)
Before this commit: robot M3Pro, 20 links, 19 joints
Joints:
- removed joint arm4_Joiint
- added joint arm4_Joint: type fixed, parent arm3, child arm4, origin xyz=0 0 0.08285 rpy=0 0 -0.027075, axis -2.6392E-05 -1 0, limit lower=-1.5708 upper=1.5708 effort=100 velocity=1
- joint arm1_Joint: type revolute -> fixed
- joint arm2_Joint: type revolute -> fixed
- joint arm3_Joint: type revolute -> fixed
- joint arm5_Joint: type revolute -> fixed
- joint llink1_Joint: type continuous -> fixed
- joint llink2_Joint: type continuous -> fixed
- joint llink3_Joint: type continuous -> fixed
- joint rlink1_Joint: type revolute -> fixed
- joint rlink2_Joint: type continuous -> fixed
- joint rlink3_Joint: type continuous -> fixed
