Commit message: update Gazebo

File: yahboomcar_ws/install/yahboom_M3Pro_description/share/yahboom_M3Pro_description/urdf/M3Pro.urdf (robot description, URDF)
Before this commit: robot M3Pro, 20 links, 19 joints
Joints:
- joint lwheel1_Joint: type revolute -> fixed
- joint lwheel2_Joint: type revolute -> fixed
- joint rwheel1_Joint: type revolute -> fixed
- joint rwheel2_Joint: type revolute -> fixed

Commit message: update Gazebo

File: yahboomcar_ws/install/yahboom_M3Pro_description/share/yahboom_M3Pro_description/urdf/M3Pro.urdf (robot description, URDF)
Before this commit: robot M3Pro, 20 links, 19 joints
Joints:
- joint arm2_Joint: origin xyz=-0.0021522 6.1185E-05 0.033 rpy=-6.3725E-05 0 -0.028422 -> xyz=-0.0021522 6.1185E-05 0.033 rpy=0.000064 -0.959931 -0.028422
- joint arm3_Joint: origin xyz=0 0 0.08285 rpy=6.3702E-05 0 0.027102 -> xyz=0 0 0.08285 rpy=1.570860 1.543631 1.570860
- joint arm4_Joint: origin xyz=0 0 0.08285 rpy=0 0 -0.027075 -> xyz=0 0 0.08285 rpy=0.000026 0.785398 -0.027064

Commit message: added ros2_control

File: yahboomcar_ws/install/yahboom_M3Pro_description/share/yahboom_M3Pro_description/urdf/M3Pro.urdf (robot description, URDF)
Before this commit: robot M3Pro, 20 links, 19 joints
Joints:
- joint lwheel1_Joint: type fixed -> revolute
- joint lwheel2_Joint: type fixed -> revolute
- joint rwheel1_Joint: type fixed -> revolute
- joint rwheel2_Joint: type fixed -> revolute

File: yahboomcar_ws/src/yahboom_M3Pro_description/urdf/M3Pro.urdf.xacro (robot description, xacro)
@@ -5,4 +5,7 @@
 <robot
   name="M3Pro">
+  xmlns:xacro="http://www.ros.org/wiki/xacro">
+  <xacro:include filename="$(find yahboom_M3Pro_description)/urdf/M3Pro.ros2_control.xacro"/>
+  <xacro:include filename="$(find yahboom_M3Pro_description)/urdf/M3Pro.gazebo.xacro"/>
   <link
     name="base_link">
@@ -884,5 +887,5 @@
   <joint
     name="lwheel1_Joint"
-    type="fixed">
+    type="continuous">
     <origin
       xyz="0.0775753787975409 0.09775 0.0399999999999998"
@@ -897,6 +900,6 @@
       lower="0"
       upper="0"
-      effort="0"
-      velocity="0" />
+      effort="10"
+      velocity="10" />
   </joint>
   <link
@@ -942,5 +945,5 @@
   <joint
     name="lwheel2_Joint"
-    type="fixed">
+    type="continuous">
     <origin
       xyz="-0.0814246212024597 0.0977499999999995 0.0399976951545867"
@@ -955,6 +958,6 @@
       lower="0"
       upper="0"
-      effort="0"
-      velocity="0" />
+      effort="10"
+      velocity="10" />
   </joint>
   <link
@@ -1000,5 +1003,5 @@
   <joint
     name="rwheel1_Joint"
-    type="fixed">
+    type="continuous">
     <origin
       xyz="0.0775753787975429 -0.0977499999999993 0.0400000000000004"
@@ -1013,6 +1016,6 @@
       lower="0"
       upper="0"
-      effort="0"
-      velocity="0" />
+      effort="10"
+      velocity="10" />
   </joint>
   <link
@@ -1058,5 +1061,5 @@
   <joint
     name="rwheel2_Joint"
-    type="fixed">
+    type="continuous">
     <origin
       xyz="-0.0814246212024577 -0.0977500000000009 0.0399976951545873"
@@ -1071,6 +1074,6 @@
       lower="0"
       upper="0"
-      effort="0"
-      velocity="0" />
+      effort="10"
+      velocity="10" />
   </joint>
   <link
@@ -1127,12 +1130,5 @@
       xyz="0 0 0" />
   </joint>
-  <gazebo>
-    <plugin name="planar_move_plugin" filename="libgazebo_ros_planar_move.so">
-      <commandTopic>cmd_vel</commandTopic>
-      <odometryTopic>odom</odometryTopic>
-      <odometryFrame>odom</odometryFrame>
-      <odometryRate>20.0</odometryRate>
-      <robotBaseFrame>base_link</robotBaseFrame>
-    </plugin>
-  </gazebo>
+<xacro:M3Pro_base_ros2_control name="GazeboSystem"/>
+<xacro:M3Pro_gazebo_ros2_control/>
 </robot>
