Commit message: update ros2_control

File: yahboomcar_ws/install/yahboom_M3Pro_description/share/yahboom_M3Pro_description/urdf/M3Pro.gazebo.xacro (robot description, xacro)
@@ -1,25 +1,14 @@
 <?xml version="1.0"?>
-<robot name="M3Pro" xmlns:xacro="http://www.ros.org/wiki/xacro">
-  <!-- Pulls in all the original SolidWorks-exported links/joints/meshes/inertials
-       untouched. We never edit M3Pro.urdf directly -- we just wrap it here. -->
-  <xacro:include filename="$(find M3Pro)/urdf/M3Pro.urdf" />
-  <!-- ===================== Gazebo materials (cosmetic only) ===================== -->
-  <gazebo reference="base_link">
-    <material>Gazebo/Grey</material>
-  </gazebo>
-  <!-- ===================== Holonomic (mecanum) drive plugin ===================== -->
-  <!-- Same idea as fake_odom_driver.py: it listens on /cmd_vel and integrates
-       (vx, vy, wz) into a pose. The difference is this now runs INSIDE Gazebo's
-       physics engine, moving the actual simulated robot body in the 3D world,
-       and publishing /odom + the odom->base_footprint TF for real. -->
-  <gazebo>
-    <plugin name="mecanum_drive_controller" filename="libgazebo_ros_planar_move.so">
-      <commandTopic>cmd_vel</commandTopic>
-      <odometryTopic>odom</odometryTopic>
-      <odometryFrame>odom</odometryFrame>
-      <odometryRate>30.0</odometryRate>
-      <robotBaseFrame>base_footprint</robotBaseFrame>
-      <broadcastTF>true</broadcastTF>
-    </plugin>
-  </gazebo>
+<robot xmlns:xacro="http://www.ros.org/wiki/xacro">
+  <xacro:macro name="M3Pro_gazebo_ros2_control" params="">
+    <gazebo>
+      <plugin name="gazebo_ros2_control" filename="libgazebo_ros2_control.so">
+        <parameters>$(find yahboom_M3Pro_description)/config/mecanum_drive_controller.yaml</parameters>
+        <ros>
+          <remapping>mecanum_drive_controller/reference_unstamped:=cmd_vel</remapping>
+          <remapping>mecanum_drive_controller/odometry:=odom</remapping>
+        </ros>
+      </plugin>
+    </gazebo>
+  </xacro:macro>
 </robot>
