Commit message: added worlds

File: yahboomcar_ws/install/yahboom_M3Pro_description/share/yahboom_M3Pro_description/urdf/M3Pro.lidar_links.xacro (robot description, xacro)
@@ -1,6 +1,7 @@
 <?xml version="1.0"?>
 <robot xmlns:xacro="http://www.ros.org/wiki/xacro">
+    <xacro:macro name="M3Pro_lidar_links" params="">
   <!-- ===== Links & Joints ===== -->
-  <link name="laser0_frame">
+    <link name="laser0_frame">
     <inertial>
       <origin xyz="0 0 0" rpy="0 0 0"/>
@@ -99,3 +100,4 @@
     </sensor>
   </gazebo>
+ </xacro:macro>
 </robot>

File: yahboomcar_ws/install/yahboom_M3Pro_description/share/yahboom_M3Pro_description/urdf/M3Pro.urdf.xacro (robot description, xacro)
@@ -1121,4 +1121,4 @@
 <xacro:M3Pro_gazebo_planar_move/>
 <xacro:M3Pro_wheel_friction/>
-<xacro:M3Pro.lidar_links/>
+<xacro:M3Pro_lidar_links/>
 </robot>
