Commit message: Restructure nav/SLAM launch files, add sim_audio, IMU and pose xacros, maze map

File: digitaltwin_ws/src/yahboom_M3Pro_description/urdf/M3Pro.camera_links.xacro (robot description, xacro)
@@ -2,5 +2,7 @@
 <robot xmlns:xacro="http://www.ros.org/wiki/xacro">
   <xacro:macro name="M3Pro_camera_links" params="">
-  <!-- Optical frame: required so image/point cloud axes match REP-103 -->
+  <!-- Color optical frame: Z forward, X right, Y down (REP-103).
+       Camera_Joint already applies rpy="1.5708 0 0", so the -π/2 roll
+       here counter-rotates back to a clean optical frame. -->
   <link name="camera_color_optical_frame"/>
   <joint name="camera_color_optical_joint" type="fixed">
@@ -9,7 +11,24 @@
     <child link="camera_color_optical_frame"/>
   </joint>
+  <!-- Depth optical frame shares the same transform as color for this sensor. -->
+  <link name="camera_depth_optical_frame"/>
+  <joint name="camera_depth_optical_joint" type="fixed">
+    <origin xyz="0 0 0" rpy="-1.5708 0 -1.5708"/>
+    <parent link="Camera"/>
+    <child link="camera_depth_optical_frame"/>
+  </joint>
+  <!-- Gazebo Harmonic RGBD camera sensor.
+       Publishes (via ros_gz_bridge):
+         /camera/color/image_raw          sensor_msgs/Image
+         /camera/depth/image_raw          sensor_msgs/Image
+         /camera/color/camera_info        sensor_msgs/CameraInfo
+         /camera/points                   sensor_msgs/PointCloud2
+       frame_id must match camera_color_optical_frame so TF resolves correctly. -->
   <gazebo reference="Camera">
-    <sensor name="camera_rgbd" type="depth">
+    <sensor name="camera_rgbd" type="rgbd_camera">
+      <topic>camera</topic>
       <update_rate>15</update_rate>
+      <always_on>true</always_on>
+      <visualize>false</visualize>
       <camera>
         <horizontal_fov>1.047</horizontal_fov>
@@ -19,24 +38,21 @@
           <format>R8G8B8</format>
         </image>
+        <depth_camera>
+          <output>depths</output>
+          <clip>
+            <near>0.1</near>
+            <far>10.0</far>
+          </clip>
+        </depth_camera>
         <clip>
           <near>0.1</near>
           <far>10.0</far>
         </clip>
+        <noise>
+          <type>gaussian</type>
+          <mean>0.0</mean>
+          <stddev>0.007</stddev>
+        </noise>
       </camera>
-      <plugin name="camera_rgbd_plugin" filename="libgazebo_ros_camera.so">
-        <ros>
-          <namespace>/camera</namespace>
-          <remapping>image_raw:=color/image_raw</remapping>
-          <remapping>camera_info:=color/camera_info</remapping>
-          <remapping>depth/image_raw:=depth/image_raw</remapping>
-          <remapping>depth/camera_info:=depth/camera_info</remapping>
-          <remapping>points:=depth/points</remapping>
-        </ros>
-        <camera_name>camera</camera_name>
-        <frame_name>camera_color_optical_frame</frame_name>
-        <hack_baseline>0.07</hack_baseline>
-        <min_depth>0.1</min_depth>
-        <max_depth>10.0</max_depth>
-      </plugin>
     </sensor>
   </gazebo>

File: digitaltwin_ws/src/yahboom_M3Pro_description/urdf/M3Pro.lidar_links.xacro (robot description, xacro)
@@ -29,7 +29,9 @@
     <child link="laser1_frame"/>
   </joint>
-  <!-- ===== Gazebo LiDAR Sensor Plugins ===== -->
+  <!-- ===== Gazebo Harmonic LiDAR Sensors ===== -->
+  <!-- Sensor data is bridged to ROS via ros_gz_bridge in gazebo_display.launch.py -->
   <gazebo reference="laser0_frame">
-    <sensor name="laser0" type="ray">
+    <sensor name="laser0" type="gpu_lidar">
+      <topic>scan0</topic>
       <pose>0 0 0 0 0 0</pose>
       <visualize>true</visualize>
@@ -55,16 +57,9 @@
         </noise>
       </ray>
-      <plugin name="laser0_plugin" filename="libgazebo_ros_ray_sensor.so">
-        <ros>
-          <namespace>/</namespace>
-          <remapping>~/out:=scan0</remapping>
-        </ros>
-        <output_type>sensor_msgs/LaserScan</output_type>
-        <frame_name>laser0_frame</frame_name>
-      </plugin>
     </sensor>
   </gazebo>
   <gazebo reference="laser1_frame">
-    <sensor name="laser1" type="ray">
+    <sensor name="laser1" type="gpu_lidar">
+      <topic>scan1</topic>
       <pose>0 0 0 0 0 0</pose>
       <visualize>true</visualize>
@@ -80,7 +75,7 @@
         </scan>
         <range>
-          <min>0.12</min>
-          <max>8.0</max>
-          <resolution>0.015</resolution>
+          <min>0.05</min>
+          <max>12.0</max>
+          <resolution>0.54</resolution>
         </range>
         <noise>
@@ -90,12 +85,4 @@
         </noise>
       </ray>
-      <plugin name="laser1_plugin" filename="libgazebo_ros_ray_sensor.so">
-        <ros>
-          <namespace>/</namespace>
-          <remapping>~/out:=scan1</remapping>
-        </ros>
-        <output_type>sensor_msgs/LaserScan</output_type>
-        <frame_name>laser1_frame</frame_name>
-      </plugin>
     </sensor>
   </gazebo>

File: digitaltwin_ws/src/yahboom_M3Pro_description/urdf/M3Pro.planar_move.xacro (robot description, xacro)
@@ -3,19 +3,17 @@
   <xacro:macro name="M3Pro_gazebo_planar_move" params="">
     <gazebo>
-      <plugin name="planar_move_plugin" filename="libgazebo_ros_planar_move.so">
-        <ros>
-          <namespace>/</namespace>
-          <remapping>cmd_vel:=cmd_vel</remapping>
-          <remapping>odom:=odom</remapping>
-        </ros>
-        <update_rate>50</update_rate>
-        <publish_rate>50</publish_rate>
-        <publish_odom>true</publish_odom>
-        <publish_odom_tf>true</publish_odom_tf>
-        <odometry_frame>odom</odometry_frame>
-        <robot_base_frame>base_link</robot_base_frame>
-        <covariance_x>0.0001</covariance_x>
-        <covariance_y>0.0001</covariance_y>
-        <covariance_yaw>0.01</covariance_yaw>
+      <plugin filename="gz-sim-diff-drive-system" name="gz::sim::systems::DiffDrive">
+        <left_joint>lwheel1_Joint</left_joint>
+        <left_joint>lwheel2_Joint</left_joint>
+        <right_joint>rwheel1_Joint</right_joint>
+        <right_joint>rwheel2_Joint</right_joint>
+        <wheel_separation>0.293</wheel_separation>
+        <wheel_radius>0.04</wheel_radius>
+        <odom_publish_frequency>50</odom_publish_frequency>
+        <topic>cmd_vel</topic>
+        <odom_topic>odom</odom_topic>
+        <tf_topic>tf</tf_topic>
+        <frame_id>odom</frame_id>
+        <child_frame_id>base_footprint</child_frame_id>
       </plugin>
     </gazebo>

File: digitaltwin_ws/src/yahboom_M3Pro_description/urdf/M3Pro.urdf.xacro (robot description, xacro)
@@ -8,6 +8,21 @@
   <xacro:include filename="$(find yahboom_M3Pro_description)/urdf/M3Pro.planar_move.xacro"/>
   <xacro:include filename="$(find yahboom_M3Pro_description)/urdf/M3Pro.camera_links.xacro"/>
+  <xacro:include filename="$(find yahboom_M3Pro_description)/urdf/M3Pro.imu.xacro"/>
   <xacro:include filename="$(find yahboom_M3Pro_description)/urdf/M3Pro.lidar_links.xacro"/>
   <xacro:include filename="$(find yahboom_M3Pro_description)/urdf/M3Pro.wheel_friction.xacro"/>
+  <xacro:include filename="$(find yahboom_M3Pro_description)/urdf/M3Pro.pose_publisher.xacro"/>
+  <!-- base_footprint is the conventional root frame used by the EKF          -->
+  <!-- (base_link_frame: base_footprint in yahboom_M3Pro_ekf.yaml) and        -->
+  <!-- matches the real robot URDF so realworld_ws bringup needs no sim hacks.-->
+  <link name="base_footprint">
+    <visual>
+      <geometry><box size="0.001 0.001 0.001"/></geometry>
+    </visual>
+  </link>
+  <joint name="link2footprint" type="fixed">
+    <parent link="base_footprint"/>
+    <child link="base_link"/>
+    <origin xyz="0 0 0" rpy="0 0 0"/>
+  </joint>
   <link
     name="base_link">
@@ -1007,5 +1022,5 @@
       link="rwheel1" />
     <axis
-      xyz="0 0 -1" />
+      xyz="0 0 1" />
     <limit
       effort="100"
@@ -1062,5 +1077,5 @@
       link="rwheel2" />
     <axis
-      xyz="0 0 -1" />
+      xyz="0 0 1" />
     <limit
       effort="100"
@@ -1111,5 +1126,5 @@
     type="fixed">
     <origin
-      xyz="0.033617 -1.0031E-05 0.0"
+      xyz="0.033617 -1.0031E-05 0.191"
       rpy="6.3751E-05 0 0" />
     <parent
@@ -1122,5 +1137,7 @@
 <xacro:M3Pro_gazebo_planar_move/>
 <xacro:M3Pro_camera_links/>
+<xacro:M3Pro_imu/>
 <xacro:M3Pro_lidar_links/>
 <xacro:M3Pro_wheel_friction/>
+<xacro:M3Pro_pose_publisher/>
 </robot>
