Commit message: added env

File: digitaltwin_ws/install/yahboom_M3Pro_description/share/yahboom_M3Pro_description/urdf/M3Pro.lidar_links.xacro (robot description, xacro)
@@ -1,103 +1 @@
-<?xml version="1.0"?>
-<robot xmlns:xacro="http://www.ros.org/wiki/xacro">
-    <xacro:macro name="M3Pro_lidar_links" params="">
-  <!-- ===== Links & Joints ===== -->
-    <link name="laser0_frame">
-    <inertial>
-      <origin xyz="0 0 0" rpy="0 0 0"/>
-      <mass value="0.0973137194820634"/>
-      <inertia ixx="4.4524583220077E-05" ixy="-1.31175451437957E-10" ixz="2.4691417638339E-09"
-               iyy="4.45241370387487E-05" iyz="-4.9776391261432E-10" izz="7.45963443980609E-05"/>
-    </inertial>
-  </link>
-  <joint name="laser0_frame_Joint" type="fixed">
-    <origin xyz="-0.11617 0.09156 0.1253" rpy="0 0 0"/>
-    <parent link="base_link"/>
-    <child link="laser0_frame"/>
-  </joint>
-  <link name="laser1_frame">
-    <inertial>
-      <origin xyz="0 0 0" rpy="0 0 0"/>
-      <mass value="0.0973137194820634"/>
-      <inertia ixx="4.4524583220077E-05" ixy="-1.31175451437957E-10" ixz="2.4691417638339E-09"
-               iyy="4.45241370387487E-05" iyz="-4.9776391261432E-10" izz="7.45963443980609E-05"/>
-    </inertial>
-  </link>
-  <joint name="laser1_frame_Joint" type="fixed">
-    <origin xyz="0.10766 -0.09078 0.1253" rpy="0 0 0"/>
-    <parent link="base_link"/>
-    <child link="laser1_frame"/>
-  </joint>
-  <!-- ===== Gazebo LiDAR Sensor Plugins ===== -->
-  <gazebo reference="laser0_frame">
-    <sensor name="laser0" type="ray">
-      <pose>0 0 0 0 0 0</pose>
-      <visualize>true</visualize>
-      <update_rate>10</update_rate>
-      <ray>
-        <scan>
-          <horizontal>
-            <samples>360</samples>
-            <resolution>1</resolution>
-            <min_angle>-3.14159</min_angle>
-            <max_angle>3.14159</max_angle>
-          </horizontal>
-        </scan>
-        <range>
-          <min>0.05</min>
-          <max>12.0</max>
-          <resolution>0.54</resolution>
-        </range>
-        <noise>
-          <type>gaussian</type>
-          <mean>0.0</mean>
-          <stddev>0.01</stddev>
-        </noise>
-      </ray>
-      <plugin name="laser0_plugin" filename="libgazebo_ros_ray_sensor.so">
-        <ros>
-          <namespace>/</namespace>
-          <remapping>~/out:=scan0</remapping>
-        </ros>
-        <output_type>sensor_msgs/LaserScan</output_type>
-        <frame_name>laser0_frame</frame_name>
-      </plugin>
-    </sensor>
-  </gazebo>
-  <gazebo reference="laser1_frame">
-    <sensor name="laser1" type="ray">
-      <pose>0 0 0 0 0 0</pose>
-      <visualize>true</visualize>
-      <update_rate>10</update_rate>
-      <ray>
-        <scan>
-          <horizontal>
-            <samples>360</samples>
-            <resolution>1</resolution>
-            <min_angle>-3.14159</min_angle>
-            <max_angle>3.14159</max_angle>
-          </horizontal>
-        </scan>
-        <range>
-          <min>0.12</min>
-          <max>8.0</max>
-          <resolution>0.015</resolution>
-        </range>
-        <noise>
-          <type>gaussian</type>
-          <mean>0.0</mean>
-          <stddev>0.01</stddev>
-        </noise>
-      </ray>
-      <plugin name="laser1_plugin" filename="libgazebo_ros_ray_sensor.so">
-        <ros>
-          <namespace>/</namespace>
-          <remapping>~/out:=scan1</remapping>
-        </ros>
-        <output_type>sensor_msgs/LaserScan</output_type>
-        <frame_name>laser1_frame</frame_name>
-      </plugin>
-    </sensor>
-  </gazebo>
- </xacro:macro>
-</robot>
+/home/pawan/yahboomcar_ws_test/digitaltwin_ws/build/yahboom_M3Pro_description/urdf/M3Pro.lidar_links.xacro

File: digitaltwin_ws/install/yahboom_M3Pro_description/share/yahboom_M3Pro_description/urdf/M3Pro.planar_move.xacro (robot description, xacro)
@@ -1,23 +1 @@
-<?xml version="1.0"?>
-<robot xmlns:xacro="http://www.ros.org/wiki/xacro">
-  <xacro:macro name="M3Pro_gazebo_planar_move" params="">
-    <gazebo>
-      <plugin name="planar_move_plugin" filename="libgazebo_ros_planar_move.so">
-        <ros>
-          <namespace>/</namespace>
-          <remapping>cmd_vel:=cmd_vel</remapping>
-          <remapping>odom:=odom</remapping>
-        </ros>
-        <update_rate>50</update_rate>
-        <publish_rate>50</publish_rate>
-        <publish_odom>true</publish_odom>
-        <publish_odom_tf>true</publish_odom_tf>
-        <odometry_frame>odom</odometry_frame>
-        <robot_base_frame>base_link</robot_base_frame>
-        <covariance_x>0.0001</covariance_x>
-        <covariance_y>0.0001</covariance_y>
-        <covariance_yaw>0.01</covariance_yaw>
-      </plugin>
-    </gazebo>
-  </xacro:macro>
-</robot>
+/home/pawan/yahboomcar_ws_test/digitaltwin_ws/build/yahboom_M3Pro_description/urdf/M3Pro.planar_move.xacro
